Commit message: feat: upgrade URDF to STL mesh visuals and rewrite README
- URDF: replace box/cylinder visuals with STL meshes for chassis,
  electronics bay, rocker arms, bogies, all 6 wheels, solar panels,
  HGA dish, LiDAR housing, mast assembly, and drill. Collision
  geometry stays as primitives for physics stability.
- Add MESH_PKG xacro property pointing to description/meshes/ pkg path
- README: full rewrite to reflect actual mission vision, working sim
  launch sequence, autonomy architecture, and engineering standards.
  Includes setup instructions, verification commands, and what-is-next.
- Commit all accumulated mesh exports, heritage models, terrain DEM
  PNG, Gazebo lpas_rover SDF model, benchmark reports, and script updates.

Co-Authored-By: Claude Sonnet 4.6 <noreply@anthropic.com>

File: ros2_ws/src/lunar_scout_description/urdf/lunar_scout.urdf.xacro (robot description, xacro)
@@ -10,4 +10,6 @@
 -->
 <robot name="lunar_scout" xmlns:xacro="http://www.ros.org/wiki/xacro">
+  <!-- STL meshes exported from NX CAD at 1:1 scale (meters) -->
+  <xacro:property name="MESH_PKG" value="package://lunar_scout_description/meshes"/>
   <!-- ============================================================
        PROPERTIES AND CONSTANTS
@@ -160,5 +162,5 @@
         <origin xyz="0 0 0" rpy="0 0 0"/>
         <geometry>
-          <box size="${rocker_length} ${rocker_width} ${rocker_height}"/>
+          <mesh filename="${MESH_PKG}/rocker_arm_${side}.stl" scale="1 1 1"/>
         </geometry>
         <material name="carbon_fiber"/>
@@ -186,5 +188,5 @@
         <origin xyz="0 0 0" rpy="${PI/2} 0 0"/>
         <geometry>
-          <cylinder radius="${wheel_radius}" length="${wheel_width}"/>
+          <mesh filename="${MESH_PKG}/wheel_assembly.stl" scale="1 1 1"/>
         </geometry>
         <material name="titanium_mesh"/>
@@ -229,5 +231,5 @@
         <origin xyz="0 0 0" rpy="0 0 0"/>
         <geometry>
-          <box size="${bogie_length} ${bogie_width} ${bogie_height}"/>
+          <mesh filename="${MESH_PKG}/bogie_arm_${side}.stl" scale="1 1 1"/>
         </geometry>
         <material name="carbon_fiber"/>
@@ -255,5 +257,5 @@
         <origin xyz="0 0 0" rpy="${PI/2} 0 0"/>
         <geometry>
-          <cylinder radius="${wheel_radius}" length="${wheel_width}"/>
+          <mesh filename="${MESH_PKG}/wheel_assembly.stl" scale="1 1 1"/>
         </geometry>
         <material name="titanium_mesh"/>
@@ -288,5 +290,5 @@
         <origin xyz="0 0 0" rpy="${PI/2} 0 0"/>
         <geometry>
-          <cylinder radius="${wheel_radius}" length="${wheel_width}"/>
+          <mesh filename="${MESH_PKG}/wheel_assembly.stl" scale="1 1 1"/>
         </geometry>
         <material name="titanium_mesh"/>
@@ -325,5 +327,5 @@
         <origin xyz="0 0 0" rpy="0 0 0"/>
         <geometry>
-          <box size="1.20 0.80 0.02"/>
+          <mesh filename="${MESH_PKG}/solar_array_panel.stl" scale="1 1 1"/>
         </geometry>
         <material name="solar_panel_blue"/>
@@ -370,5 +372,5 @@
       <origin xyz="0 0 0" rpy="0 0 0"/>
       <geometry>
-        <box size="${chassis_length} ${chassis_width} ${chassis_height}"/>
+        <mesh filename="${MESH_PKG}/chassis_body.stl" scale="1 1 1"/>
       </geometry>
       <material name="aluminum_gold"/>
@@ -387,5 +389,5 @@
       <origin xyz="0 0 0" rpy="0 0 0"/>
       <geometry>
-        <box size="0.50 0.80 0.30"/>
+        <mesh filename="${MESH_PKG}/electronics_bay.stl" scale="1 1 1"/>
       </geometry>
       <material name="white_thermal"/>
@@ -440,5 +442,5 @@
       <origin xyz="0 0 0" rpy="0 0 0"/>
       <geometry>
-        <cylinder radius="0.051" length="0.072"/>
+        <mesh filename="${MESH_PKG}/lidar_housing.stl" scale="1 1 1"/>
       </geometry>
       <material name="sensor_black"/>
@@ -465,5 +467,5 @@
       <origin xyz="0 0 0" rpy="0 0 0"/>
       <geometry>
-        <box size="0.04 0.04 0.35"/>
+        <mesh filename="${MESH_PKG}/mast_assembly.stl" scale="1 1 1"/>
       </geometry>
       <material name="carbon_fiber"/>
@@ -600,10 +602,9 @@
        ============================================================ -->
   <link name="hga_link">
-    <!-- Parabolic dish approximated as cylinder + cone -->
     <xacro:cylinder_inertia m="1.2" r="0.22" h="0.05"/>
     <visual>
       <origin xyz="0 0 0" rpy="0 0 0"/>
       <geometry>
-        <cylinder radius="0.22" length="0.05"/>
+        <mesh filename="${MESH_PKG}/hga_dish.stl" scale="1 1 1"/>
       </geometry>
       <material name="antenna_white"/>
@@ -637,5 +638,5 @@
       <origin xyz="0 0 -0.30" rpy="0 0 0"/>
       <geometry>
-        <cylinder radius="0.04" length="0.60"/>
+        <mesh filename="${MESH_PKG}/drill_assembly.stl" scale="1 1 1"/>
       </geometry>
       <material name="science_gray"/>

File: ros2_ws/src/lunar_scout_description/urdf/nasa_heritage_meshes.xacro (robot description, xacro)
@@ -1,4 +1,130 @@
 <?xml version="1.0"?>
 <robot xmlns:xacro="http://www.ros.org/wiki/xacro">
-<!-- NASA heritage model mesh references — auto-generated -->
+<!-- NASA heritage model mesh references � auto-generated -->
+  <!-- Heritage: Curiosity Rover Body (NASA-3D-Resources) -->
+  <xacro:macro name="chassis_body_heritage_mesh" params="">
+    <visual>
+      <geometry>
+        <mesh filename="package://lunar_scout_description/meshes/chassis_body.stl"
+              scale="1 1 1"/>
+      </geometry>
+    </visual>
+    <collision>
+      <geometry>
+        <mesh filename="package://lunar_scout_description/meshes/chassis_body.stl"/>
+      </geometry>
+    </collision>
+  </xacro:macro>
+  <!-- Heritage: Curiosity ChemCam (NASA-3D-Resources) -->
+  <xacro:macro name="nav_cam_assembly_heritage_mesh" params="">
+    <visual>
+      <geometry>
+        <mesh filename="package://lunar_scout_description/meshes/nav_cam_assembly.stl"
+              scale="1 1 1"/>
+      </geometry>
+    </visual>
+    <collision>
+      <geometry>
+        <mesh filename="package://lunar_scout_description/meshes/nav_cam_assembly.stl"/>
+      </geometry>
+    </collision>
+  </xacro:macro>
+  <!-- Heritage: Curiosity RTG (enclosure geometry only) (NASA-3D-Resources) -->
+  <xacro:macro name="electronics_bay_heritage_mesh" params="">
+    <visual>
+      <geometry>
+        <mesh filename="package://lunar_scout_description/meshes/electronics_bay.stl"
+              scale="1 1 1"/>
+      </geometry>
+    </visual>
+    <collision>
+      <geometry>
+        <mesh filename="package://lunar_scout_description/meshes/electronics_bay.stl"/>
+      </geometry>
+    </collision>
+  </xacro:macro>
+  <!-- Heritage: Curiosity Wheels (NASA-3D-Resources) -->
+  <xacro:macro name="wheel_assembly_heritage_mesh" params="">
+    <visual>
+      <geometry>
+        <mesh filename="package://lunar_scout_description/meshes/wheel_assembly.stl"
+              scale="1 1 1"/>
+      </geometry>
+    </visual>
+    <collision>
+      <geometry>
+        <mesh filename="package://lunar_scout_description/meshes/wheel_assembly.stl"/>
+      </geometry>
+    </collision>
+  </xacro:macro>
+  <!-- Heritage: Curiosity HGA (NASA-3D-Resources) -->
+  <xacro:macro name="hga_dish_heritage_mesh" params="">
+    <visual>
+      <geometry>
+        <mesh filename="package://lunar_scout_description/meshes/hga_dish.stl"
+              scale="1 1 1"/>
+      </geometry>
+    </visual>
+    <collision>
+      <geometry>
+        <mesh filename="package://lunar_scout_description/meshes/hga_dish.stl"/>
+      </geometry>
+    </collision>
+  </xacro:macro>
+  <!-- Heritage: Curiosity Mast (NASA-3D-Resources) -->
+  <xacro:macro name="nav_cam_assembly_heritage_mesh" params="">
+    <visual>
+      <geometry>
+        <mesh filename="package://lunar_scout_description/meshes/nav_cam_assembly.stl"
+              scale="1 1 1"/>
+      </geometry>
+    </visual>
+    <collision>
+      <geometry>
+        <mesh filename="package://lunar_scout_description/meshes/nav_cam_assembly.stl"/>
+      </geometry>
+    </collision>
+  </xacro:macro>
+  <!-- Heritage: Curiosity Rocker (NASA-3D-Resources) -->
+  <xacro:macro name="rocker_arm_left_heritage_mesh" params="">
+    <visual>
+      <geometry>
+        <mesh filename="package://lunar_scout_description/meshes/rocker_arm_left.stl"
+              scale="1 1 1"/>
+      </geometry>
+    </visual>
+    <collision>
+      <geometry>
+        <mesh filename="package://lunar_scout_description/meshes/rocker_arm_left.stl"/>
+      </geometry>
+    </collision>
+  </xacro:macro>
+  <!-- Heritage: Curiosity Bogie (NASA-3D-Resources) -->
+  <xacro:macro name="bogie_arm_left_heritage_mesh" params="">
+    <visual>
+      <geometry>
+        <mesh filename="package://lunar_scout_description/meshes/bogie_arm_left.stl"
+              scale="1 1 1"/>
+      </geometry>
+    </visual>
+    <collision>
+      <geometry>
+        <mesh filename="package://lunar_scout_description/meshes/bogie_arm_left.stl"/>
+      </geometry>
+    </collision>
+  </xacro:macro>
+  <!-- Heritage: Curiosity Solar Panel (NASA-3D-Resources) -->
+  <xacro:macro name="solar_array_panel_heritage_mesh" params="">
+    <visual>
+      <geometry>
+        <mesh filename="package://lunar_scout_description/meshes/solar_array_panel.stl"
+              scale="1 1 1"/>
+      </geometry>
+    </visual>
+    <collision>
+      <geometry>
+        <mesh filename="package://lunar_scout_description/meshes/solar_array_panel.stl"/>
+      </geometry>
+    </collision>
+  </xacro:macro>
 </robot>
